Commit message: Home upper joints to the saved pose on every stack startup
Use bounded Stanford stop homing for motors 1 and 2, preserve the stop-derived frame, and hold the saved upper home. Keep wheel hubs passive until operator-aligned live capture. Add the required agent workflow, checked launcher, target consistency checks, and pose history.

Validated ROS Jazzy build, C++ homing checks, 19 calibration tests, expanded URDF targets, and confirmation guard. Pi installation and live saved-home check remain pending after SSH connectivity was lost.

File: ros2_ws/src/pupper_v3_description/description/components.xacro (robot description, xacro)
@@ -2,4 +2,8 @@
 <robot xmlns:xacro="http://www.ros.org/wiki/xacro">
     <xacro:macro name="define_components">
+        <!-- The homing_* values below are legacy hanging-pose fallback values.
+             Normal real hardware now uses startup_upper_home: stop homing and
+             saved targets for motors 1/2, raw passive hubs with manual capture.
+             See STARTUP_UPPER_HOME.md; old no-stop upper-leg comments are historical. -->
         <joint name="leg_front_r_1">
             <param name="can_channel">2</param>

File: ros2_ws/src/pupper_v3_description/description/pupper_v3.ros2_control.xacro (robot description, xacro)
@@ -3,7 +3,17 @@
     <xacro:include filename="$(find pupper_v3_description)/description/components.xacro" />
     <xacro:macro name="pupper_v3_system">
+        <xacro:property name="upper_home" value="${xacro.load_yaml('$(find pupper_v3_description)/description/upper_home.yaml')}" />
         <ros2_control name="control_board_hardware_interface" type="system">
             <hardware>
                 <plugin>control_board_hardware_interface/ControlBoardHardwareInterface</plugin>
+                <param name="startup_upper_home">true</param>
+                <param name="upper_home_leg_front_r_1">${upper_home['leg_front_r_1']}</param>
+                <param name="upper_home_leg_front_r_2">${upper_home['leg_front_r_2']}</param>
+                <param name="upper_home_leg_front_l_1">${upper_home['leg_front_l_1']}</param>
+                <param name="upper_home_leg_front_l_2">${upper_home['leg_front_l_2']}</param>
+                <param name="upper_home_leg_back_r_1">${upper_home['leg_back_r_1']}</param>
+                <param name="upper_home_leg_back_r_2">${upper_home['leg_back_r_2']}</param>
+                <param name="upper_home_leg_back_l_1">${upper_home['leg_back_l_1']}</param>
+                <param name="upper_home_leg_back_l_2">${upper_home['leg_back_l_2']}</param>
                 <!-- <param name="use_imu">false</param> -->
             </hardware>
