Commit message: Revert Stanford stop-homing for motors 1/2: no real hard stop on this leg
67e3857 reintroduced Stanford-style stop-seeking homing for the upper
joints, but never ran on real hardware before tonight (its own message
notes the Pi install/live check were pending). Three live attempts all
failed differently: leg_back_l_1 frozen at exact zero, then a two-leg
no-stop drift, then a "Homing speed exceeded" abort.

The seek assumes a genuine mechanical stop exists to detect a torque
spike against -- but 95dc175 already established (MuJoCo droop-pose
analysis, verified against photos of the leg hanging free) that this
leg design has none, for exactly this reason: driving toward a
nonexistent stop just goes until something incidental gets in the way,
which is what the live failures show. Falls back to the gravity-droop
homing path, which just ran clean and instant on hardware (all 8
joints homed, front/back sanity checks agree within ~1 deg).

Co-Authored-By: Claude Sonnet 5 <noreply@anthropic.com>

File: ros2_ws/src/pupper_v3_description/description/components.xacro (robot description, xacro)
@@ -2,8 +2,4 @@
 <robot xmlns:xacro="http://www.ros.org/wiki/xacro">
     <xacro:macro name="define_components">
-        <!-- The homing_* values below are legacy hanging-pose fallback values.
-             Normal real hardware now uses startup_upper_home: stop homing and
-             saved targets for motors 1/2, raw passive hubs with manual capture.
-             See STARTUP_UPPER_HOME.md; old no-stop upper-leg comments are historical. -->
         <joint name="leg_front_r_1">
             <param name="can_channel">2</param>

File: ros2_ws/src/pupper_v3_description/description/pupper_v3.ros2_control.xacro (robot description, xacro)
@@ -3,17 +3,7 @@
     <xacro:include filename="$(find pupper_v3_description)/description/components.xacro" />
     <xacro:macro name="pupper_v3_system">
-        <xacro:property name="upper_home" value="${xacro.load_yaml('$(find pupper_v3_description)/description/upper_home.yaml')}" />
         <ros2_control name="control_board_hardware_interface" type="system">
             <hardware>
                 <plugin>control_board_hardware_interface/ControlBoardHardwareInterface</plugin>
-                <param name="startup_upper_home">true</param>
-                <param name="upper_home_leg_front_r_1">${upper_home['leg_front_r_1']}</param>
-                <param name="upper_home_leg_front_r_2">${upper_home['leg_front_r_2']}</param>
-                <param name="upper_home_leg_front_l_1">${upper_home['leg_front_l_1']}</param>
-                <param name="upper_home_leg_front_l_2">${upper_home['leg_front_l_2']}</param>
-                <param name="upper_home_leg_back_r_1">${upper_home['leg_back_r_1']}</param>
-                <param name="upper_home_leg_back_r_2">${upper_home['leg_back_r_2']}</param>
-                <param name="upper_home_leg_back_l_1">${upper_home['leg_back_l_1']}</param>
-                <param name="upper_home_leg_back_l_2">${upper_home['leg_back_l_2']}</param>
                 <!-- <param name="use_imu">false</param> -->
             </hardware>
